File: kicad/DAC7718.kicad_sch (KiCad schematic)
At the start: 32 parts, among them U5 REF5025AD, U8 REF5025AD, U9 DAC7718

Commit message: added gain calc pdfs
Parts:
- removed C25, C27: 1uF, Capacitor_SMD:C_0402_1005Metric_Pad0.74x0.62mm_HandSolder, symbol Device:C
- removed D3: D_Schottky, symbol Device:D_Schottky
- removed JP1: Jumper_2_Open, Resistor_SMD:R_0201_0603Metric, symbol Jumper:Jumper_2_Open
- removed R12, R8, R9: 10k, Resistor_SMD:R_0402_1005Metric_Pad0.72x0.64mm_HandSolder, symbol Device:R
- removed U8: REF5025AD, Package_SO:VSSOP-8_3.0x3.0mm_P0.65mm, symbol Reference_Voltage:REF5025AD
- added JP1, JP3, JP4: Jumper_2_Small_Open, symbol Jumper:Jumper_2_Small_Open
- added JP2: Jumper_2_Small_Bridged, symbol Jumper:Jumper_2_Small_Bridged
- added NT1, NT2: NetTie_2, symbol Device:NetTie_2
- added NT3, NT5: NetTie_3, symbol Device:NetTie_3
- added NT4: NetTie_4, symbol Device:NetTie_4
- added TP3: TestPoint, symbol Connector:TestPoint
- added U6: DG611E, ThinMiniQFN:ThinMiniQFN-16_2.6mm_1.8mm, symbol DG61x:DG611E
- C12: value 22uF -> 10uF
- C17: value 1uF -> 10uF
- C6: value 1uF -> 100nF
Connections:
- net +5V: now also NT2.1, U6.1 (S1), U6.11 (V+), U6.12 (S2); no longer C6.1
- net AVDD: now also U6.13 (D2)
- net AVSS: now also C12.1, C6.2, U6.8 (D3); no longer C17.2
- net DAC_CLR: now also R7.1; no longer R6.1
- net DAC_LDAC: now also R1.1, JP4.2 (B); no longer R5.1
- net DAC_RST: now also R4.1; no longer R3.1
- net DAC_SPI_CS: now also R2.1; no longer R1.1
- net DAC_WAKEUP: now also R3.1; no longer R2.1
- net DGND: now also C10.1, C28.2, C29.2, JP1.1 (A), JP2.1 (A), JP4.1 (A), NT1.2, NT4.1
- net DVDD: now also U6.16 (D1)
- net GND: now also C17.2, C6.1, NT1.1, NT5.2, U6.2 (V-), U6.3 (GND); no longer C10.2, C28.2, C29.2, C6.2
- net IOVDD: now also C10.2, JP3.2 (B), NT2.2; no longer R6.2
- net REFA: now also NT3.1; no longer C11.1, D2.2 (A), U5.6 (Vout)
- net REFB: now also NT3.3; no longer C12.1
- net at U9.29 (GPIO-1): now also NT4.4
- net at U9.30 (GPIO-0): now also NT4.3
- net at U9.19 (GPIO-2): now also NT4.2
- net at U9.3 (AIN-0): now also NT5.1
- net at U9.46 (AIN-1): now also NT5.3
- net DAC_RSTSEL: no longer names the net of U9.51 (RSTSEL)
- net DAC_RSTSEL: now also R5.1, JP1.2 (B); no longer R4.1
- net DAC_USB_BTC: no longer names the net of U9.50 (~{USB/BTC})
- net DAC_USB_BTC: now also R6.1, JP2.2 (B); no longer R7.1
- net dac_monitor: no longer names the net of C26.2, U9.14 (VMON)
- net dac_monitor: now also TP3.1
- new net: C11.1, D2.2 (A), U5.6 (Vout), U6.4 (S4)
- new net: NT3.2, U6.5 (D4)
- new net: JP3.1 (A), R6.2
- new net -5V: U6.9 (S3)
- new net AVDD_ENABLE: U6.14 (IN2), U6.7 (IN3)
- new net DVDD_ENABLE: U6.15 (IN1)
- new net VREF_ENABLE: U6.6 (IN4)
- no-connect marks 4 -> 1
Other:
- note added: "DAC7718 Datasheet"
- note added: "DAC7718 Eval Board User Guide"
- note added: "For gain calcuations, see "doc/design/DAC7718 Gain - SCE Disabled.pdf""
- note added: "RSTSEL: V_{OUT} = 0v or V_{OUT} = -Fullscale (join JP1+JP3 and cut JP2)"
- note added: "The power should be applied in the order: - IOVDD - DVDD - AVDD/AVSS - reference voltage"
- note added: "~{CLR}: All V_{out} pins connected to A_{GND}"
- note added: "~{CS}: SPI bus chip select"
- note added: "~{LDAC}: Update DAC outputs. Join JP4 for async mode."
- note added: "~{WAKEUP}: Restore SPI from sleep mode"
- note removed: "Connect this is if only one REF5025 populated"
- moved on the sheet: C11, C13, C14, C26, C28, C29, C5, C7, D2, R1, R2, R3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
