File: kicad/PSU.kicad_sch (KiCad schematic)
At the start: 8 parts, among them J6 Barrel_Jack_Switch, U2 TLV75801PDBV, U6 DG611E

Commit message: added gain calc pdfs
Parts:
- removed C24: 100nF, Capacitor_SMD:C_0402_1005Metric_Pad0.74x0.62mm_HandSolder, symbol Device:C
- removed NT1: NetTie_2, symbol Device:NetTie_2
- removed R17: 10k, Resistor_SMD:R_0402_1005Metric_Pad0.72x0.64mm_HandSolder, symbol Device:R
- removed U6: DG611E, ThinMiniQFN:ThinMiniQFN-16_2.6mm_1.8mm, symbol DG61x:DG611E
Connections:
- net 3V3_ENABLE is gone; now on net +5V: U2.3 (EN)
- no-connect marks 3 -> 1
Other:
- moved on the sheet: J6, R26, R27, U2
