File: kicad/Tiny4xPoweredStereoMixer.kicad_sch (KiCad schematic)
At the start: 31 parts, among them J1 AudioJack3_SwitchTR, J2 AudioJack3_SwitchTR, J3 AudioJack3_SwitchTR, J4 AudioJack3_SwitchTR, J6 Barrel_Jack_Switch, J9 AudioJack3_SwitchTR, U5 TL074

Commit message: saving work in progress
Parts:
- removed C8, C9: 100nF, Capacitor_SMD:C_0402_1005Metric_Pad0.74x0.62mm_HandSolder, symbol Device:C
- removed J1, J2, J3, J4, J9: AudioJack3_SwitchTR, Connector_Audio:Jack_3.5mm_CUI_SJ1-3535NG_Horizontal, symbol Connector_Audio:AudioJack3_SwitchTR
- removed J6: Barrel_Jack_Switch, Connector_BarrelJack:BarrelJack_Horizontal, symbol Connector:Barrel_Jack_Switch
- removed R1, R10, R12, R13, R14, R15, R2, R3, R4, R5, R6, R7, R8, R9: 10k, Resistor_SMD:R_0402_1005Metric_Pad0.72x0.64mm_HandSolder, symbol Device:R
- removed RV1, RV2, RV3, RV4: 10k, Potentiometers:Alps_RK12L12_Double_Horizontal, symbol Device:R_Potentiometer_Dual_Separate
- removed U5: TL074, SOT-23-THIN-14:SOIC-14, symbol Amplifier_Operational:TL074
- added J5: AudioJack3_SwitchTR, Connector_Audio:Jack_3.5mm_CUI_SJ1-3535NG_Horizontal, symbol Connector_Audio:AudioJack3_SwitchTR
Connections:
- net GND: now also J5.RN, J5.S, J5.TN
- new net VCA_SSI2164/ch5_left_audio: J5.T
- new net VCA_SSI2164/ch5_right_audio: J5.R
- no-connect marks 0 -> 1
Other:
- removed sheet LM1117 Low Dropout Regulator
- removed sheet TPS54202 Inverting PSU
- added sheet AUDIO_INPUT (AUDIO_INPUT.kicad_sch)
- added sheet DAC7718 (DAC7718.kicad_sch)
- added sheet PSU (PSU.kicad_sch)
- added sheet ROTARY_ENCODERS (ROTARY_ENCODERS.kicad_sch)
- added sheet VCA_SSI2164 (VCA_SSI2164.kicad_sch)
- added sheet mcu (mcu.kicad_sch)
- note removed: "Bridge unless populated if AC coupling is needed"
- note removed: "Min input for TPS54202 = 4.5V"
- moved on the sheet: H1, H2, H3, H4

Commit message: added gain calc pdfs
Other:
- sheet mcu renamed ESP32-S3
- sheet DAC7718 ports: added AVDD_ENABLE, DVDD_ENABLE, VREF_ENABLE; removed DAC_RSTSEL, DAC_USB_BTC, dac_monitor
- sheet ESP32-S3 ports: added VREF_ENABLE; removed 3V3_ENABLE, AVSS_ENABLE, DAC_RSTSEL, DAC_USB_BTC, IOVDD_ENABLE
- sheet PSU ports: added none; removed 3V3_ENABLE, AVDD_ENABLE, AVSS_ENABLE, DVDD_ENABLE, IOVDD_ENABLE
- moved on the sheet: J5
