File: kicad/mcu.kicad_sch (KiCad schematic)
At the start: 6 parts, among them J7 USB_B_Micro, U1 ESP32-S3-WROOM-1

Commit message: added gain calc pdfs
Parts:
- added C24, C32, C33: 100nF, symbol Device:C
- added C25: 1uF, symbol Device:C
- added C27: 22uF, symbol Device:C
- added NT6, NT7, NT8: NetTie_2, symbol Device:NetTie_2
- added R9: 10K, symbol Device:R
- added SW5, SW6: SW_SPST, symbol Switch:SW_SPST
Connections:
- net +3.3V: now also C24.1, C27.1, R9.1
- net DAC_SPI_CLK: now also NT8.1; no longer U1.20 (IO12)
- net DAC_SPI_CS: now also NT6.1; no longer U1.18 (IO10)
- net DAC_SPI_MOSI: now also NT7.1; no longer U1.19 (IO11)
- net BOOT_GPIO0: now reaches U1.27 (IO0)
- net BOOT_GPIO0: now also C33.1, SW6.2 (B)
- net ENABLE renamed CHIP_PUP
- net CHIP_PUP: now also C25.1, C32.1, R9.2, SW5.2 (B)
- net GND renamed DGND
- net DGND: now also C24.2, C25.2, C27.2, C32.2, C33.2, SW5.1 (A), SW6.1 (A)
- new net FSPICLK: NT8.2, U1.20 (IO12)
- new net FSPIQ: NT7.2, U1.19 (IO11)
- new net FSPIWP: NT6.2, U1.18 (IO10)
- no-connect marks 5 -> 32
Other:
- note added: "ESP32-S3 datasheet"
- note added: "ESP32-S3-DevKitC-1_V1.1 Schematic"
- note added: "ESP32-S3-WROOM-1 datasheet"
- note added: "ESPS3 PCNT ======== https://github.com/espressif/esp-idf/tree/v5.3.2/ examples/peripherals/pcnt/rotary_encoder"
- note added: "ESPS3 SPI ======= https://github.com/espressif/esp-idf/tree/v5.3.2/ examples/peripherals/spi_master/lcd"
- note added: "JTAG SETUP: ======== https://docs.espressif.com/projects/ esp-idf/en/stable/esp32s3/api-guides/ jtag-debugging/configure-builtin-jtag.html"
- note added: "Power Sequencing =========== See DAC7118 sheet"
- note removed: "ESPS3 PCNT ========== https://github.com/espressif/esp-idf/tree/v5.3.2/ examples/peripherals/pcnt/rotary_encoder"
- note removed: "ESPS3 SPI ========= https://github.com/espressif/esp-idf/tree/v5.3.2/ examples/peripherals/spi_master/lcd"
- note removed: "JTAG SETUP: =========== https://docs.espressif.com/projects/ esp-idf/en/stable/esp32s3/api-guides/ jtag-debugging/configure-builtin-jtag.html"
- moved on the sheet: D4, D5, D6, D7, J7, U1
