File: kicad/tps54202_inverting_psu.kicad_sch (KiCad schematic)
At the start: 18 parts, among them U1 TPS54202DDC

Commit message: saving work in progress
Parts:
- renumbered C4 to C1, C7 to C15, C9 to C16, C1 to C18, C26 to C19, C5 to C2, C24 to C20, C25 to C21, C2 to C22, C3 to C23, C6 to C3, C8 to C4, R2 to R16, R3 to R18, R4 to R19, U1 to U3
Connections:
- net TPS54202_ENABLE: now reaches U3.5 (EN)
- no-connect marks 1 -> 0

Commit message: added gain calc pdfs
Changed lines of the file:
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@@
-	)
-	(junction
-		(at 71.12 109.22)
-		(diameter 0)
-		(color 0 0 0 0)
 	)
 	(junction
@@
 					(unit 1)
 				)
-			)
-		)
-	)
-	(symbol
-		(lib_id "power:PWR_FLAG")
-		(at 71.12 109.22 180)
-		(unit 1)
-		(exclude_from_sim no)
-		(in_bom yes)
-		(on_board yes)
-		(dnp no)
-		(fields_autoplaced yes)
-		(property "Reference" "#FLG02"
-			(at 71.12 111.125 0)
-			(effects
-				(font
-					(size 1.27 1.27)
-				)
-				(hide yes)
-			)
-		)
-		(property "Value" "PWR_FLAG"
-			(at 71.12 114.3 0)
-			(effects
-				(font
-					(size 1.27 1.27)
-				)
-			)
-		)
-		(property "Footprint" ""
-			(at 71.12 109.22 0)
-			(effects
-				(font
-					(size 1.27 1.27)
-				)
-				(hide yes)
-			)
-		)
-		(property "Datasheet" "~"
-			(at 71.12 109.22 0)
-			(effects
-				(font
-					(size 1.27 1.27)
-				)
-				(hide yes)
-			)
-		)
-		(property "Description" "Special symbol for telling ERC where power comes from"
-			(at 71.12 109.22 0)
-			(effects
-				(font
-					(size 1.27 1.27)
-				)
-				(hide yes)
-			)
-		)
-		(pin "1"
-		)
-		(instances
-			(project "Tiny4xPoweredStereoMixer"
-				(path "/68c4b081-ef47-4ba5-a55f-4ef66cb2b598/90ba425d-eaf5-48b4-804f-91b46c159bdf/2de80bd8-59cf-45da-b027-4f047eba247b"
-					(reference "#FLG02")
-					(unit 1)
-				)
